File: Day_09_DGCFT/001/001.kicad_pcb (KiCad board)
At the start: 2 copper layers, 88 x 97.8 mm, 26 parts, among them J1 CONN_01X03, J2 CONN_01X03, J3 CONN_02X03, J4 CONN_01X02, J5 CONN_01X02, U1 ATTINY85-20SU, U2 LM340MP-5.0/NOPB

Commit message: Update
Parts:
- removed LED7, LED8: WS2812B, Granabot_Footprints:WS2812B
- D1: moved to B.Cu
- moved J1 41.6 mm to (115.6, 95.2)
- moved LED5 41.0 mm to (153.7, 92.7)
- moved J2 39.9 mm to (148.0, 95.2), turned to 0 degrees
- moved D1 36.4 mm to (163.8, 102.2)
- moved R1 33.1 mm to (163.8, 108.0)
- moved C3 20.7 mm to (151.8, 113.0), turned to 0 degrees
- moved J3 16.2 mm to (115.6, 108.6), turned to 270 degrees
- moved LED4 15.5 mm to (133.3, 135.3)
- moved U1 12.3 mm to (130.8, 95.9), turned to 0 degrees
- moved D2 10.5 mm to (141.0, 118.7), turned to 180 degrees
- moved LED6 9.96 mm to (153.7, 125.1)
- moved LED3 9.71 mm to (107.3, 125.1)
- moved C2 8.82 mm to (151.8, 118.7), turned to 0 degrees
- moved J4 8.03 mm to (146.1, 127.6)
- moved LED1 7.96 mm to (133.3, 78.7)
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Connections:
- LED6 pad 4: Net-(LED6-Pad4) -> (no net)
Routing:
- net MISO-1-PWM: track 0.00 -> 5.91 mm, vias 0 -> 1
- added copper zone on B.Cu, net GND
- added copper zone on F.Cu, net GND
Other:
- board text added: "#Makevember"
- board text added: "Day 9"
